File: bttoken.brd (EAGLE design)
At the start: 84.5 x 33.5 mm, 53 parts, among them IC1 0, Q1 32k, T1 MMBT3904, X1 FCI-MICRO-USB

Commit message: Auto routing works
Parts:
- moved U$13 1.01 mm to (9.42, 21.2), turned to 0 degrees
- moved U$1 0.89 mm to (24.5, 12.1), turned to 225 degrees

Commit message: A little optimization
Parts:
- moved D1 53.1 mm to (1.65, 7.68), turned to 90 degrees
- moved T1 34.1 mm to (7.36, 7.86)
- moved C4 30.1 mm to (11.8, 6.80)
- moved R12 22.9 mm to (34.6, 1.73), turned to 180 degrees
- moved C10 7.84 mm to (11.7, 2.67), turned to 270 degrees
- moved LED_CHRG 2.85 mm to (58.8, 7.71)
- moved R2 2.32 mm to (57.4, 2.13)
- moved C12 2.16 mm to (39.1, 1.64)
- moved C9 1.81 mm to (16.9, 1.78)
- moved IC1 1.59 mm to (52.8, 7.08)
- moved JP1 0.89 mm to (27.2, 1.78)

Commit message: New revision with moved quartz, changed filter, etc. Broke autorouting
Parts:
- IC1: device adafruit:TO92 -> DonB:SOT23
- U$13: value BR-LE4.0-S3 -> BR-LE4.0-S3-NC; device BlueRadios_D2_S2_C46_Eagle_footprint:BR-LE4.0-X2A -> BlueRadios_D2_S2_C46_Eagle_footprint:BR-LE4.0-X2A-NC
- moved Q1 80.7 mm to (2.46, 10.2), turned to 180 degrees
- moved T1 28.5 mm to (32.9, 20.6)
- moved D1 23.0 mm to (2.90, 30.6)
- moved C4 19.2 mm to (28.1, 16.9)
- moved C10 16.7 mm to (28.1, 5.87)
- moved U$1 10.2 mm to (15.8, 6.76), turned to 315 degrees
- moved C9 9.62 mm to (25.6, 5.87), turned to 270 degrees
- moved PZO_HDR 2.37 mm to (38.4, 17.4)
- moved U$13 2.03 mm to (11.4, 21.7)
- moved S1 1.24 mm to (59.7, 28.8)
- moved X1 0.50 mm to (76.1, 1.86)
- moved BAT1 0.36 mm to (71.3, 16.3)
Connections:
- net GND: now also U$13.P$11
- net VBAT: now also IC1.3; no longer IC1.2
- net VCC: now also IC1.2; no longer IC1.3

Commit message: Checkpoint
Parts:
- moved Q1 61.8 mm to (62.6, 24.6)
- moved C1 50.0 mm to (8.89, 40.4)
- moved JP1 46.3 mm to (61.7, 32.7)
- moved R5 38.9 mm to (63.8, 38.8)
- moved R12 36.5 mm to (25.7, 37.1)
- moved C14 35.2 mm to (74.3, 11.9), turned to 0 degrees
- moved LED_CHRG 33.9 mm to (49.8, 40.4)
- moved R7 33.5 mm to (72.2, 38.8)
- moved C8 33.3 mm to (57.1, 22.6), turned to 180 degrees
- moved U$1 33.0 mm to (48.4, 12.3), turned to 225 degrees
- moved C9 31.8 mm to (57.3, 8.89), turned to 90 degrees
- moved S1 31.2 mm to (81.6, 6.61)
- moved C7 31.1 mm to (57.3, 18.5), turned to 0 degrees
- moved C15 30.5 mm to (74.3, 8.18), turned to 0 degrees
- moved C10 29.2 mm to (57.3, 3.91), turned to 90 degrees
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Routing:
- net VBAT: track 0.00 -> 119.1 mm, vias 0 -> 3
- net BTH_RST: track 0.00 -> 52.1 mm, vias 0 -> 2
- net VBUS: track 0.00 -> 50.1 mm
- net VCC: track 0.00 -> 49.2 mm
- net BTH_SEL: track 0.00 -> 44.9 mm, vias 0 -> 2
- net SPI_CLK: track 0.00 -> 44.9 mm, vias 0 -> 2
- net SPI_MISO: track 0.00 -> 44.7 mm, vias 0 -> 2
- net SPI_MOSI: track 0.00 -> 44.0 mm, vias 0 -> 2
- net N$1: track 0.00 -> 16.9 mm
- net XT2IN: track 0.00 -> 13.9 mm
- net N$9: track 0.00 -> 11.7 mm
- net XT2OUT: track 0.00 -> 10.3 mm
- net IR_CTL: track 0.00 -> 10.1 mm
- net N$13: track 0.00 -> 7.40 mm
- net PZO1: track 0.00 -> 4.46 mm
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Other:
- board size 84.5 x 33.5 mm -> 92.3 x 45.4 mm
